Commit message: add gr1t1 mujoco sim

File: model/GR1T1/urdf/GR1T1.urdf (robot description, URDF)
Before this commit: robot GR1T1, 37 links, 36 joints
Links:
- added link base, mass 6.45116957899581; collision cylinder length=0.29 radius=0.039; visual mesh filename=package://gr1t1_description/meshes/base.STL
- link dummy_link: mass 6.45116957899581 -> None; geometry 
Joints:
- added joint dummy_link_to_base: type fixed, parent dummy_link, child base, origin xyz=0 0 0 rpy=0 0 0
- joint l_foot_heel_joint: origin xyz=-0.0445 0 -0.042 rpy=0 0 0 -> xyz=-0.0445 0 -0.05 rpy=0 0 0
- joint l_foot_toe_joint: origin xyz=0.1415 0 -0.042 rpy=0 0 0 -> xyz=0.1415 0 -0.05 rpy=0 0 0
- joint l_hip_roll: parent dummy_link -> base
- joint r_foot_heel_joint: origin xyz=-0.0445 0 -0.042 rpy=0 0 0 -> xyz=-0.0445 0 -0.05 rpy=0 0 0
- joint r_foot_toe_joint: origin xyz=0.1415 0 -0.042 rpy=0 0 0 -> xyz=0.1415 0 -0.05 rpy=0 0 0
- joint r_hip_roll: parent dummy_link -> base
- joint waist_yaw: parent dummy_link -> base
